File: 02-hardware/esc_brushless/microcontroller.sch (KiCad schematic (older format))
At the start: 0 parts

Commit message: Schematics v1.0 - Architecture V1.0, fix DRC issues
Parts:
- added C27, C28, C29: 2.2u, p_Package_Capacitor_SMD:C_0603_1608Metric_Pad1.08x0.95mm_HandSolder, symbol p_Passive:C_0603
- added Q7: BC848B, p_Package_SOT:SOT-23, symbol p_Transistor_bipolar:BC848B
- added R37: DNP, p_Package_Resistor_SMD:R_0603_1608Metric_Pad0.98x0.95mm_HandSolder, symbol p_Passive:R_0603
- added R38, R40, R41: R_0603, p_Package_Resistor_SMD:R_0603_1608Metric_Pad0.98x0.95mm_HandSolder, symbol p_Passive:R_0603
- added TP1, TP2: test_point, p_Package_Misc:TP_SMD_1.25mm, symbol p_Misc:test_point
- added U2: STM32G030_C8, p_Package_QFP:LQFP-48_7x7mm_P0.5mm, symbol p_MCU:STM32G030_C8
Connections:
- new net: TP1.1 (TP), U2.34 (PA12)
- new net: TP2.1 (TP), U2.37 (PA15)
- new net: Q7.2 (B), R38.1, R40.2
- new net 3.3V_MCU: C27.1, C28.1, C29.1, R41.2, U2.4 (VBAT), U2.5 (VREF+), U2.6 (VDD/VDDA)
- new net ADC_A: U2.21 (PB2)
- new net ADC_B: U2.20 (PB1)
- new net ADC_C: U2.19 (PB0)
- new net ADC_PVDD: U2.22 (PB10)
- new net DC_CAL: U2.31 (PC7)
- new net EN_GATE: U2.30 (PC6)
- new net GND: C27.2, C28.2, C29.2, Q7.1 (E), R40.1, U2.7 (VSS/VSSA)
- new net INH_A: U2.28 (PA8)
- new net INH_B: U2.29 (PA9)
- new net INH_C: U2.32 (PA10)
- new net INL_A: U2.25 (PB13)
- new net INL_B: U2.26 (PB14)
- new net INL_C: U2.27 (PB15)
- new net LED: U2.1 (PC13)
- new net PWM: Q7.3 (C), R37.2, R41.1, U2.33 (PA11)
- new net PWM_IN: R37.1, R38.2
- new net RS485_DE: U2.3 (PC15)
- new net SO1: U2.11 (PA0)
- new net SO2: U2.12 (PA1)
- new net SPI_CS: U2.15 (PA4), U2.17 (PA6)
- new net SPI_MOSI: U2.18 (PA7)
- new net SPI_SCK: U2.16 (PA5)
- new net SW_CLK: U2.36 (PA14)
- new net SW_DIO: U2.35 (PA13)
- new net TEMP_SENSOR1: U2.23 (PB11)
- new net TEMP_SENSOR2: U2.24 (PB12)
- new net UART_RX: U2.46 (PB7)
- new net UART_TX: U2.45 (PB6)
- new net \FLT: U2.40 (PD2)
- new net \MCU_RST: U2.42 (PB3)
- new net \OVR_CUR_FLT: U2.39 (PD1)
- new net \PWRGD_FLT: U2.38 (PD0)
- new net \RS485_RE: U2.2 (PC14)
- no-connect marks 0 -> 10
