File: 02-hardware/esc_brushless/microcontroller.sch (KiCad schematic (older format))
At the start: 11 parts, among them Q7 BC848B, U2 STM32G030_C8

Commit message: Schematics v1.0 - PCB layout v1.0
Parts:
- removed TP2: test_point, p_Package_Misc:TP_SMD_1.25mm, symbol p_Misc:test_point
Connections:
- net TEMP_SENSOR2 is gone; now on net SO1: U2.24 (PB12)
- net ADC_A: now also U2.19 (PB0); no longer U2.21 (PB2)
- net ADC_C: now also U2.21 (PB2); no longer U2.19 (PB0)
- net ADC_PVDD: now also U2.11 (PA0); no longer U2.22 (PB10)
- net DC_CAL: now also U2.34 (PA12); no longer U2.31 (PC7)
- net EN_GATE: now also U2.33 (PA11); no longer U2.30 (PC6)
- net INH_A: now also U2.32 (PA10); no longer U2.28 (PA8)
- net INH_C: now also U2.28 (PA8); no longer U2.32 (PA10)
- net INL_A: now also U2.27 (PB15); no longer U2.25 (PB13)
- net INL_C: now also U2.25 (PB13); no longer U2.27 (PB15)
- net LED: now also U2.18 (PA7); no longer U2.1 (PC13)
- net PWM: now also U2.37 (PA15); no longer U2.33 (PA11)
- net RS485_DE: now also U2.16 (PA5); no longer U2.3 (PC15)
- net SO1: no longer U2.11 (PA0)
- net SO2: now also U2.23 (PB11); no longer U2.12 (PA1)
- net SPI_CS: now also U2.45 (PB6); no longer U2.15 (PA4), U2.17 (PA6)
- net SPI_MOSI: now also U2.44 (PB5); no longer U2.18 (PA7)
- net SPI_SCK: now also U2.42 (PB3); no longer U2.16 (PA5)
- net TEMP_SENSOR1: now also U2.22 (PB10); no longer U2.23 (PB11)
- net UART_RX: now also U2.14 (PA3); no longer U2.46 (PB7)
- net UART_TX: now also U2.13 (PA2); no longer U2.45 (PB6)
- net \FLT: now also U2.48 (PB9); no longer U2.40 (PD2)
- net \MCU_RST: now also U2.38 (PD0); no longer U2.42 (PB3)
- net \OVR_CUR_FLT: now also U2.47 (PB8); no longer U2.39 (PD1)
- net \PWRGD_FLT: now also U2.46 (PB7); no longer U2.38 (PD0)
- net \RS485_RE: now also U2.15 (PA4); no longer U2.2 (PC14)
- net at TP1.1 (TP): now also U2.41 (PD3); no longer U2.34 (PA12)
- net SPI_MISO: now reaches U2.43 (PB4)
- no-connect marks 10 -> 11
Other:
- moved on the sheet: TP1
Changed lines of the file:
@@
 SPI_MISO
 Text HLabel 2150 2300 0    50   Input ~ 0
-SO1
+SO2
 Text HLabel 2150 1050 0    50   UnSpc ~ 0
 REF
 Text HLabel 2150 2400 0    50   Input ~ 0
-SO2
+SO1
 Text HLabel 9900 4350 2    50   Output ~ 0
 DC_CAL
@@
 Text HLabel 2150 1350 0    50   Output ~ 0
 UART_TX
-$Comp
-L p_MCU:STM32G030_C8 U2
-U 1 1 607AAEF6
-P 6150 3600
-F 0 "U2" H 6150 5315 50  0000 C CNN
-F 1 "STM32G030_C8" H 6150 5224 50  0000 C CNN
-F 2 "p_Package_QFP:LQFP-48_7x7mm_P0.5mm" H 6250 1950 50  0001 C CNN
-F 3 "" H 6100 2800 50  0001 C CNN
-	1    6150 3600
-	1    0    0    -1
-$EndComp
 Wire Wire Line
 	5450 2250 5300 2250
@@
 3.3V_MCU
 Wire Wire Line
-	6850 3150 7500 3150
-Wire Wire Line
-	6850 3250 7500 3250
-Text Label 7500 3250 0    50   ~ 0
+	5450 2750 4800 2750
+Wire Wire Line
+	5450 2850 4800 2850
+Text Label 4800 2850 2    50   ~ 0
 UART1_RX
 Wire Wire Line
@@
 	2150 3850 5450 3850
 Wire Wire Line
-	5450 3150 4550 3150
-Text Label 4550 3150 0    50   ~ 0
+	6850 2950 7750 2950
+Text Label 7750 2950 2    50   ~ 0
 SPI_MISO
 Wire Wire Line
-	5450 3250 4550 3250
-Text Label 4550 3250 0    50   ~ 0
+	6850 3050 7750 3050
+Text Label 7750 3050 2    50   ~ 0
 SPI_MOSI
 Wire Wire Line
-	5450 2950 4550 2950
-Text Label 4550 2950 0    50   ~ 0
-SPI_SS
-Wire Wire Line
-	5450 3050 4550 3050
-Text Label 4550 3050 0    50   ~ 0
+	6850 3150 7500 3150
+Wire Wire Line
+	6850 2850 7750 2850
+Text Label 7750 2850 2    50   ~ 0
 SPI_SCK
 Wire Wire Line
@@
 	5300 2350 5300 2250
 Connection ~ 5300 2250
-Text Label 4550 2950 0    50   ~ 0
-SPI_MISO
-Wire Wire Line
-	6850 3850 7500 3850
-Text Label 7500 3850 0    50   ~ 0
-TIM_CH1N
 Wire Wire Line
 	6850 3950 7500 3950
-Text Label 7500 3950 0    50   ~ 0
-TIM_CH2N
-Wire Wire Line
-	6850 4050 7500 4050
-Text Label 7500 4050 0    50   ~ 0
-TIM_CH3N
 Text HLabel 9900 3350 2    50   Output ~ 0
 INH_A
@@
 INL_C
 Text Label 9000 3350 0    50   ~ 0
-TIM_CH1
+TIM_CH3
 Text Label 9000 3450 0    50   ~ 0
-TIM_CH1N
+TIM_CH3N
 Text Label 9000 3550 0    50   ~ 0
 TIM_CH2
@@
 TIM_CH2N
 Text Label 9000 3750 0    50   ~ 0
-TIM_CH3
+TIM_CH1
 Text Label 9000 3850 0    50   ~ 0
-TIM_CH3N
+TIM_CH1N
 Wire Wire Line
 	9000 3350 9900 3350
@@
 	2150 900  5300 900
 Wire Wire Line
-	5450 2550 5200 2550
-Wire Wire Line
-	5200 2550 5200 2300
-Wire Wire Line
-	5200 2300 2150 2300
-Wire Wire Line
-	2150 2400 5100 2400
-Wire Wire Line
-	5100 2400 5100 2650
-Wire Wire Line
-	5100 2650 5450 2650
+	2150 2400 3300 2400
 Wire Wire Line
 	2150 2200 3300 2200
@@
 ADC_IN9
 Text Label 3300 2200 0    50   ~ 0
-ADC_IN8
+ADC_IN10
 Wire Wire Line
 	2150 2000 3300 2000
@@
 	2150 1900 3300 1900
 Text Label 3300 1900 0    50   ~ 0
-ADC_IN11
+ADC_IN2
 Text Label 3300 2000 0    50   ~ 0
-ADC_IN10
+ADC_IN8
 Wire Wire Line
 	2150 1800 3300 1800
 Text Label 3300 1800 0    50   ~ 0
-ADC_IN12
+ADC_IN11
 Text Label 3300 2400 0    50   ~ 0
-ADC_IN1
+ADC_IN16
 Text Label 3300 2300 0    50   ~ 0
-ADC_IN0
-Wire Wire Line
-	6850 3650 7500 3650
-Wire Wire Line
-	6850 3550 7500 3550
-Text Label 7500 3550 0    50   ~ 0
-ADC_IN11
-Text Label 7500 3650 0    50   ~ 0
-ADC_IN12
+ADC_IN15
+Text Label 4550 2550 0    50   ~ 0
+ADC_IN2
+Text Label 7750 2550 2    50   ~ 0
+ADC_IN8
 Wire Wire Line
 	6850 2750 7500 2750
@@
 ADC_IN10
 Wire Wire Line
-	6850 2550 7500 2550
-Text Label 7500 2550 0    50   ~ 0
-ADC_IN8
-Wire Wire Line
 	2150 1050 2800 1050
 Text Label 2800 1050 0    50   ~ 0
@@
 Text Label 3300 3200 0    50   ~ 0
 \PWRGD_FLT
-Wire Wire Line
-	6850 4250 7500 4250
-Text Label 7500 4250 0    50   ~ 0
-\PWRGD_FLT
-Wire Wire Line
-	6850 4350 7500 4350
-Text Label 7500 4350 0    50   ~ 0
+Text Label 7500 3350 0    50   ~ 0
 \OVR_CUR_FLT
 Wire Wire Line
-	6850 4450 7500 4450
-Text Label 7500 4450 0    50   ~ 0
+	5450 2950 4800 2950
+Text Label 7500 3450 0    50   ~ 0
 \FLT
 Text Label 9000 4250 0    50   ~ 0
@@
 Wire Wire Line
 	9000 4950 9900 4950
-Text Label 4550 3650 0    50   ~ 0
-PWM
-Wire Wire Line
-	4550 3650 5450 3650
 Wire Wire Line
 	4550 3550 5450 3550
@@
 TIM_CH3
 Wire Wire Line
-	4550 4250 5450 4250
-Wire Wire Line
-	4550 4350 5450 4350
-Wire Wire Line
-	4550 4450 5450 4450
-Wire Wire Line
-	4550 4550 5450 4550
-Wire Wire Line
-	4550 4650 5450 4650
-Text Label 4550 4250 0    50   ~ 0
+	4550 3750 5450 3750
+Wire Wire Line
+	4550 3250 5450 3250
+Text Label 4800 3650 2    50   ~ 0
 EN_GATE
-Text Label 4550 4350 0    50   ~ 0
+Text Label 4550 3750 0    50   ~ 0
 DC_CAL
-Text Label 4550 4450 0    50   ~ 0
+Text Label 4550 3250 0    50   ~ 0
 LED
-Text Label 4550 4550 0    50   ~ 0
-\RS485_RE
-Text Label 4550 4650 0    50   ~ 0
-RS485_DE
 $Comp
 L p_Transistor_bipolar:BC848B Q7
@@
 Wire Wire Line
 	2150 5500 2400 5500
-Text HLabel 9900 2850 2    50   Output ~ 0
+Text HLabel 9900 4750 2    50   Output ~ 0
 \MCU_RST
 Wire Wire Line
-	9900 2850 6850 2850
+	9900 4750 9000 4750
 Text HLabel 9900 5200 2    50   UnSpc ~ 0
 GND
@@
 Wire Wire Line
 	9750 5200 9750 5300
-$Comp
-L p_Misc:test_point TP2
-U 1 1 608E544E
-P 5100 4050
-F 0 "TP2" H 4900 4050 50  0000 C CNN
-F 1 "test_point" H 5087 4184 50  0001 C CNN
-F 2 "p_Package_Misc:TP_SMD_1.25mm" H 5100 3850 50  0001 C CNN
-F 3 "" H 5100 4050 50  0001 C CNN
-	1    5100 4050
-	1    0    0    -1
-$EndComp
 Wire Wire Line
 	2150 3950 5450 3950
-Wire Wire Line
-	5200 4050 5450 4050
 $Comp
 L p_Misc:test_point TP1
 U 1 1 609117C2
-P 5100 3750
-F 0 "TP1" H 4900 3750 50  0000 C CNN
-F 1 "test_point" H 5087 3884 50  0001 C CNN
-F 2 "p_Package_Misc:TP_SMD_1.25mm" H 5100 3550 50  0001 C CNN
-F 3 "" H 5100 3750 50  0001 C CNN
-	1    5100 3750
-	1    0    0    -1
-$EndComp
-Wire Wire Line
-	5200 3750 5450 3750
+P 7200 4550
+F 0 "TP1" H 7000 4550 50  0000 C CNN
+F 1 "test_point" H 7187 4684 50  0001 C CNN
+F 2 "p_Package_Misc:TP_SMD_1.25mm" H 7200 4350 50  0001 C CNN
+F 3 "" H 7200 4550 50  0001 C CNN
+	1    7200 4550
+	-1   0    0    1
+$EndComp
+Wire Wire Line
+	7100 4550 6850 4550
 NoConn ~ 5450 4850
 Wire Wire Line
-	6850 3750 7500 3750
-Text Label 7500 3750 0    50   ~ 0
+	6850 3450 7500 3450
+Text Label 4800 2750 2    50   ~ 0
+UART1_TX
+Text Label 4800 4050 2    50   ~ 0
+PWM
+Wire Wire Line
+	5450 4050 4800 4050
+Wire Wire Line
+	4550 2550 5450 2550
+Wire Wire Line
+	7750 2550 6850 2550
+Wire Wire Line
+	7500 3250 6850 3250
+Wire Wire Line
+	7500 3350 6850 3350
+Text Label 4800 2950 2    50   ~ 0
+\RS485_RE
+NoConn ~ 5450 4550
+NoConn ~ 5450 4650
+Text Label 7500 3150 0    50   ~ 0
+SPI_SS
+Wire Wire Line
+	7750 3550 6850 3550
+Text Label 7750 3550 2    50   ~ 0
+ADC_IN11
+Text Label 7500 3250 0    50   ~ 0
+\PWRGD_FLT
+Text Label 7500 3950 0    50   ~ 0
+TIM_CH2N
+Wire Wire Line
+	4800 3650 5450 3650
+NoConn ~ 5450 4450
+NoConn ~ 6850 4450
+Text Label 4800 3050 2    50   ~ 0
+RS485_DE
+Wire Wire Line
+	5450 3050 4800 3050
+Text Label 7500 4050 0    50   ~ 0
+TIM_CH3N
+Wire Wire Line
+	6850 4050 7500 4050
+Text Label 7500 3850 0    50   ~ 0
+TIM_CH1N
+Wire Wire Line
+	6850 3850 7500 3850
+NoConn ~ 5450 4350
+NoConn ~ 6850 4850
+Wire Wire Line
+	3300 2300 2150 2300
+Wire Wire Line
+	6850 3750 8000 3750
+Text Label 8000 3750 0    50   ~ 0
 ADC_IN16
-Text HLabel 2150 1700 0    50   Input ~ 0
-TEMP_SENSOR2
-Wire Wire Line
-	2150 1700 3300 1700
-Text Label 3300 1700 0    50   ~ 0
-ADC_IN16
-NoConn ~ 6850 4550
-NoConn ~ 6850 4750
-NoConn ~ 6850 4850
-NoConn ~ 5450 2750
-NoConn ~ 5450 2850
-Text Label 7500 3150 0    50   ~ 0
-UART1_TX
-NoConn ~ 6850 2950
-NoConn ~ 6850 3050
-NoConn ~ 6850 3350
-NoConn ~ 6850 3450
+Text Label 8000 3650 0    50   ~ 0
+ADC_IN15
+Wire Wire Line
+	8000 3650 6850 3650
+$Comp
+L p_MCU:STM32G030_C8 U2
+U 1 1 607AAEF6
+P 6150 3600
+F 0 "U2" H 6150 5315 50  0000 C CNN
+F 1 "STM32G030_C8" H 6150 5224 50  0000 C CNN
+F 2 "p_Package_QFP:LQFP-48_7x7mm_P0.5mm" H 6250 1950 50  0001 C CNN
+F 3 "" H 6100 2800 50  0001 C CNN
+	1    6150 3600
+	1    0    0    -1
+$EndComp
+NoConn ~ 5450 2650
+NoConn ~ 5450 4250
+Text Label 9000 4750 0    50   ~ 0
+\MCU_RST
+Wire Wire Line
+	6850 4250 7750 4250
+Text Label 7750 4250 2    50   ~ 0
+\MCU_RST
+NoConn ~ 5450 3150
+NoConn ~ 6850 4350
 $EndSCHEMATC
