File: 02-hardware/esc_brushless/mos_drive_stage.sch (KiCad schematic (older format))
At the start: 1 part

Commit message: Schematics v1.0 - Architecture V1.0, fix DRC issues
Parts:
- removed U?: DRV8301, p_Package_SO:HTSSOP-56-1EP_6.1x14mm_P0.5mm_EP3.61x6.35mm.kicad_mod, symbol p_Driver_IC:DRV8301
- added C10, C9: 47u, p_Package_Capacitor_SMD:C_1210_3225Metric_Pad1.33x2.70mm_HandSolder, symbol p_Passive:C_1210
- added C11, C12, C17, C25, C26: 4.7u, p_Package_Capacitor_SMD:C_0603_1608Metric_Pad1.08x0.95mm_HandSolder, symbol p_Passive:C_0603
- added C13, C14, C15, C16: 1u, p_Package_Capacitor_SMD:C_0603_1608Metric_Pad1.08x0.95mm_HandSolder, symbol p_Passive:C_0603
- added C18, C19, C20, C21: 100n, p_Package_Capacitor_SMD:C_0603_1608Metric_Pad1.08x0.95mm_HandSolder, symbol p_Passive:C_0603
- added C22: 22n, p_Package_Capacitor_SMD:C_0603_1608Metric_Pad1.08x0.95mm_HandSolder, symbol p_Passive:C_0603
- added C23: 2.2u, p_Package_Capacitor_SMD:C_0603_1608Metric_Pad1.08x0.95mm_HandSolder, symbol p_Passive:C_0603
- added C24: 47u, p_Package_Capacitor_SMD:C_1206_3216Metric_Pad1.33x1.80mm_HandSolder, symbol p_Passive:C_1206
- added D2: MBRS260T3G, p_Package_Diode_SMD:D_SMB_Handsoldering, symbol p_Diode:MBRS260T3G
- added L1: 22u, p_Package_Inductor_SMD:SDR0805, symbol p_Passive:L_SDR0805
- added R26, R27, R28, R29, R30, R31, R32, R33, R34, R35: 10k, p_Package_Resistor_SMD:R_0603_1608Metric_Pad0.98x0.95mm_HandSolder, symbol p_Passive:R_0603
- added U1: DRV8301, p_Package_SO:HTSSOP-56-1EP_6.1x14mm_P0.5mm_EP3.61x6.35mm, symbol p_Driver_IC:DRV8301
Connections:
- new net: R32.1, U1.1 (RT_CLK)
- new net: R27.1, U1.7 (DTC)
- new net: C15.1, U1.23 (DVDD)
- new net: C22.1, U1.14 (CP1)
- new net: C22.2, U1.15 (CP2)
- new net: C16.1, U1.27 (AVDD)
- new net: C23.2, U1.13 (GVDD)
- new net: C19.2, U1.43 (BST_B)
- new net: C18.2, U1.48 (BST_A)
- new net: C20.2, U1.38 (BST_C)
- new net: C21.1, D2.1 (K), L1.1, U1.50 (PH), U1.51 (PH)
- new net: C25.1, R35.2
- new net: C17.1, U1.56 (SS_TR)
- new net: C21.2, U1.52 (BST_BK)
- new net: R33.2, R34.1, U1.3 (VSENSE)
- new net: R29.1, U1.25 (SO1)
- new net: R30.1, U1.26 (SO2)
- new net +3V3: R26.1, R28.2, R31.1, U1.49 (VDD_SPI)
- new net +5V: C24.1, L1.2, R33.1
- new net DC_CAL: U1.12 (DC_CAL)
- new net EN_GATE: U1.16 (EN_GATE)
- new net GH_A: U1.47 (GH_A)
- new net GH_B: U1.42 (GH_B)
- new net GH_C: U1.37 (GH_C)
- new net GL_A: U1.45 (GL_A)
- new net GL_B: U1.40 (GL_B)
- new net GL_C: U1.35 (GL_C)
- new net GND: C10.2, C11.2, C12.2, C13.2, C14.2, C17.2, C23.1, C24.2, C25.2, C26.2, C9.2, D2.2 (A), R27.2, R32.2, R34.2, U1.57 (GND_EP)
- new net GNDA: C15.2, C16.2, U1.28 (AGND)
- new net INH_A: U1.17 (INH_A)
- new net INH_B: U1.19 (INH_B)
- new net INH_C: U1.21 (INH_C)
- new net INL_A: U1.18 (INL_A)
- new net INL_B: U1.20 (INL_B)
- new net INL_C: U1.22 (INL_C)
- new net REF: U1.24 (REF)
- new net SH_A: C18.1, U1.46 (SH_A)
- new net SH_B: C19.1, U1.41 (SH_B)
- new net SH_C: C20.1, U1.36 (SH_C)
- new net SL_A: U1.44 (SL_A)
- new net SL_B: U1.39 (SL_B)
- new net SL_C: U1.34 (SL_C)
- new net SN1: U1.33 (SN1)
- new net SN2: U1.31 (SN2)
- new net SO1: C13.1, R29.2
- new net SO2: C14.1, R30.2
- new net SP1: U1.32 (SP1)
- new net SP2: U1.30 (SP2)
- new net SPI_CLK: U1.11 (SCLK)
- new net SPI_CS: U1.8 (nSCS)
- new net SPI_MISO: U1.10 (SDO)
- new net SPI_MOSI: U1.9 (SDI)
- new net V_PWR: C10.1, C11.1, C12.1, C9.1, U1.29 (PVDD1), U1.53 (PVDD2), U1.54 (PVDD2)
- new net \FLT: R28.1, U1.6 (nFAULT)
- new net \OVR_CUR_FLT: R26.2, U1.5 (nOCTW)
- new net \PWRGD_FLT: R31.2, U1.4 (PWRGD)
- new net comp: C26.1, R35.1, U1.2 (COMP)
- no-connect marks 0 -> 1
