File: 02-hardware/esc_brushless/RS488_phy.sch (KiCad schematic (older format))
At the start: 2 parts

Commit message: Schematics v1.0 - Fix DRC issues
Parts:
- gave numbers to parts that had none: 2
Other:
- moved on the sheet: C34, U4
Changed lines of the file:
@@
 $Descr A4 11693 8268
 encoding utf-8
-Sheet 7 6
+Sheet 6 6
 Title "ESC Brushless - CAN phy"
 Date "2021-03-10"
@@
 Comment4 ""
 $EndDescr
-Text HLabel 2400 2000 0    50   Input ~ 0
+Text HLabel 3850 2800 0    50   UnSpc ~ 0
 5_VCC
-Text HLabel 2400 2800 0    50   Input ~ 0
+Text HLabel 3850 3600 0    50   Input ~ 0
 \RS485_RE
-Text HLabel 2400 2900 0    50   Output ~ 0
+Text HLabel 3850 3700 0    50   Output ~ 0
 RS485_RX
-Text HLabel 7150 2900 2    50   BiDi ~ 0
+Text HLabel 8600 3700 2    50   BiDi ~ 0
 RS485-A
-Text HLabel 7150 3200 2    50   BiDi ~ 0
+Text HLabel 8600 4000 2    50   BiDi ~ 0
 RS485-B
 Wire Wire Line
-	5100 2900 7150 2900
+	6550 3700 8600 3700
 Wire Wire Line
-	7150 3200 5100 3200
+	8600 4000 6550 4000
 $Comp
-L p_Passive:C_0603 C?
+L p_Passive:C_0603 C34
 U 1 1 609345BE
-P 2900 2250
-F 0 "C?" H 3015 2296 50  0000 L CNN
-F 1 "100n" H 3015 2205 50  0000 L CNN
-F 2 "p_Package_Capacitor_SMD:C_0603_1608Metric_Pad1.08x0.95mm_HandSolder" H 2900 2250 50  0001 C CNN
-F 3 "" H 2900 2250 50  0001 C CNN
-	1    2900 2250
+P 4350 3050
+F 0 "C34" H 4465 3096 50  0000 L CNN
+F 1 "100n" H 4465 3005 50  0000 L CNN
+F 2 "p_Package_Capacitor_SMD:C_0603_1608Metric_Pad1.08x0.95mm_HandSolder" H 4350 3050 50  0001 C CNN
+F 3 "" H 4350 3050 50  0001 C CNN
+	1    4350 3050
 	1    0    0    -1
 $EndComp
 Wire Wire Line
-	2900 2100 2900 2000
+	4350 2900 4350 2800
 $Comp
-L power:GND #PWR?
+L power:GND #PWR056
 U 1 1 609345C5
-P 2900 2450
-F 0 "#PWR?" H 2900 2200 50  0001 C CNN
-F 1 "GND" H 2900 2300 50  0000 C CNN
-F 2 "" H 2900 2450 50  0001 C CNN
-F 3 "" H 2900 2450 50  0001 C CNN
-	1    2900 2450
+P 4350 3250
+F 0 "#PWR056" H 4350 3000 50  0001 C CNN
+F 1 "GND" H 4350 3100 50  0000 C CNN
+F 2 "" H 4350 3250 50  0001 C CNN
+F 3 "" H 4350 3250 50  0001 C CNN
+	1    4350 3250
 	1    0    0    -1
 $EndComp
 Wire Wire Line
-	2900 2400 2900 2450
+	4350 3200 4350 3250
 Wire Wire Line
-	2400 2000 2900 2000
-Connection ~ 2900 2000
+	3850 2800 4350 2800
+Connection ~ 4350 2800
 $Comp
-L power:GND #PWR?
+L power:GND #PWR057
 U 1 1 6093530A
-P 5200 3450
-F 0 "#PWR?" H 5200 3200 50  0001 C CNN
-F 1 "GND" H 5205 3277 50  0000 C CNN
-F 2 "" H 5200 3450 50  0001 C CNN
-F 3 "" H 5200 3450 50  0001 C CNN
-	1    5200 3450
+P 6650 4250
+F 0 "#PWR057" H 6650 4000 50  0001 C CNN
+F 1 "GND" H 6655 4077 50  0000 C CNN
+F 2 "" H 6650 4250 50  0001 C CNN
+F 3 "" H 6650 4250 50  0001 C CNN
+	1    6650 4250
 	1    0    0    -1
 $EndComp
 Wire Wire Line
-	5200 3300 5200 3450
-Text HLabel 2400 4150 0    50   UnSpc ~ 0
+	6650 4100 6650 4250
+Text HLabel 3850 4950 0    50   UnSpc ~ 0
 GND
 $Comp
-L power:GND #PWR?
+L power:GND #PWR055
 U 1 1 60935C2E
-P 2550 4250
-F 0 "#PWR?" H 2550 4000 50  0001 C CNN
-F 1 "GND" H 2555 4077 50  0000 C CNN
-F 2 "" H 2550 4250 50  0001 C CNN
-F 3 "" H 2550 4250 50  0001 C CNN
-	1    2550 4250
+P 4000 5050
+F 0 "#PWR055" H 4000 4800 50  0001 C CNN
+F 1 "GND" H 4005 4877 50  0000 C CNN
+F 2 "" H 4000 5050 50  0001 C CNN
+F 3 "" H 4000 5050 50  0001 C CNN
+	1    4000 5050
 	1    0    0    -1
 $EndComp
 Wire Wire Line
-	2400 4150 2550 4150
+	3850 4950 4000 4950
 Wire Wire Line
-	2550 4250 2550 4150
+	4000 5050 4000 4950
 $Comp
-L p_Driver_IC:MAX487CSA_ESA U?
+L p_Driver_IC:MAX487CSA_ESA U4
 U 1 1 604A635F
-P 4750 3050
-F 0 "U?" H 4550 3500 50  0000 C CNN
-F 1 "MAX487CSA_ESA" H 4750 2650 50  0000 C CNN
-F 2 "p_Package_SO:SOIC-8_3.9x4.9mm_P1.27mm" H 4750 3050 50  0001 C CNN
-F 3 "${KI_PERSO_COMPLIB}/datasheets/p_Driver_IC/MAX488.pdf" H 4750 3050 50  0001 C CNN
-	1    4750 3050
+P 6200 3850
+F 0 "U4" H 6000 4300 50  0000 C CNN
+F 1 "MAX487CSA_ESA" H 6200 3450 50  0000 C CNN
+F 2 "p_Package_SO:SOIC-8_3.9x4.9mm_P1.27mm" H 6200 3850 50  0001 C CNN
+F 3 "${KI_PERSO_COMPLIB}/datasheets/p_Driver_IC/MAX488.pdf" H 6200 3850 50  0001 C CNN
+	1    6200 3850
 	1    0    0    -1
 $EndComp
 Wire Wire Line
-	5100 3300 5200 3300
+	6550 4100 6650 4100
 Wire Wire Line
-	5450 2800 5450 2000
+	6900 3600 6900 2800
 Wire Wire Line
-	2900 2000 5450 2000
-Wire Wire Line
-	5100 2800 5450 2800
-Text HLabel 2400 3200 0    50   Input ~ 0
+	4350 2800 6900 2800
+Text HLabel 3850 4000 0    50   Input ~ 0
 RS485_DE
 Wire Wire Line
-	2400 2800 4400 2800
+	3850 3600 5850 3600
 Wire Wire Line
-	2400 3200 4400 3200
+	3850 4000 5850 4000
 Wire Wire Line
-	2400 2900 4400 2900
-Text HLabel 2400 3300 0    50   Input ~ 0
+	3850 3700 5850 3700
+Text HLabel 3850 4100 0    50   Input ~ 0
 RS485_TX
 Wire Wire Line
-	2400 3300 4400 3300
+	3850 4100 5850 4100
+Wire Wire Line
+	6550 3600 6900 3600
 $EndSCHEMATC
